File: Apple-1 ROM_RAM.kicad_pcb (KiCad board)
At the start: 2 copper layers, 103 x 53.5 mm, 6 parts, among them J1 Conn_02x22_Apple_1-Connector_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, T1 Jumper, U1 2732, U2 2732

Commit message: Add files via upload
Parts:
- moved T1 91.2 mm to (117.5, 132.6)
Routing:
- net /T: track 5.75 -> 163.4 mm, vias 0 -> 1
- net Net-(T1-Pad1): track 150.6 -> 20.7 mm
Other:
- board text added: "S Address to U1"
- board text added: "T Address to U2"
Changed lines of the file:
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@@
   (general
     (thickness 1.6)
-    (drawings 9)
-    (tracks 208)
+    (drawings 11)
+    (tracks 212)
     (zones 0)
     (modules 6)
@@
       (drillshape 0)
       (scaleselection 1)
-      (outputdirectory "C:/Users/garyr/OneDrive/Documents/Vintage computers/Projects/Apple-1 ROM_RAM/Gerber/"))
+      (outputdirectory "Gerber/"))
   )
   (net 0 "")
@@
     (add_net "Net-(T1-Pad1)")
   )
+  (module Connector_PinHeader_2.54mm:PinHeader_1x02_P2.54mm_Vertical (layer F.Cu)
+    (at 117.5262 132.60746)
+    (descr "Through hole straight pin header, 1x02, 2.54mm pitch, single row")
+    (tags "Through hole pin header THT 1x02 2.54mm single row")
+    (fp_text reference T1 (at 0 -2.33) (layer F.SilkS)
+      (effects (font (size 1 1) (thickness 0.15)))
+    )
+    (fp_text value Jumper (at 0 4.87) (layer F.Fab)
+      (effects (font (size 1 1) (thickness 0.15)))
+    )
+    (fp_line (start -0.635 -1.27) (end 1.27 -1.27) (layer F.Fab) (width 0.1))
+    (fp_line (start 1.27 -1.27) (end 1.27 3.81) (layer F.Fab) (width 0.1))
+    (fp_line (start 1.27 3.81) (end -1.27 3.81) (layer F.Fab) (width 0.1))
+    (fp_line (start -1.27 3.81) (end -1.27 -0.635) (layer F.Fab) (width 0.1))
+    (fp_line (start -1.27 -0.635) (end -0.635 -1.27) (layer F.Fab) (width 0.1))
+    (fp_line (start -1.33 3.87) (end 1.33 3.87) (layer F.SilkS) (width 0.12))
+    (fp_line (start -1.33 1.27) (end -1.33 3.87) (layer F.SilkS) (width 0.12))
+    (fp_line (start 1.33 1.27) (end 1.33 3.87) (layer F.SilkS) (width 0.12))
+    (fp_line (start -1.33 1.27) (end 1.33 1.27) (layer F.SilkS) (width 0.12))
+    (fp_line (start -1.33 0) (end -1.33 -1.33) (layer F.SilkS) (width 0.12))
+    (fp_line (start -1.33 -1.33) (end 0 -1.33) (layer F.SilkS) (width 0.12))
+    (fp_line (start -1.8 -1.8) (end -1.8 4.35) (layer F.CrtYd) (width 0.05))
+    (fp_line (start -1.8 4.35) (end 1.8 4.35) (layer F.CrtYd) (width 0.05))
+    (fp_line (start 1.8 4.35) (end 1.8 -1.8) (layer F.CrtYd) (width 0.05))
+    (fp_line (start 1.8 -1.8) (end -1.8 -1.8) (layer F.CrtYd) (width 0.05))
+    (fp_text user %R (at 0 1.27 90) (layer F.Fab)
+      (effects (font (size 1 1) (thickness 0.15)))
+    )
+    (pad 1 thru_hole rect (at 0 0) (size 1.7 1.7) (drill 1) (layers *.Cu *.Mask)
+      (net 46 "Net-(T1-Pad1)"))
+    (pad 2 thru_hole oval (at 0 2.54) (size 1.7 1.7) (drill 1) (layers *.Cu *.Mask)
+      (net 44 /T))
+    (model ${KISYS3DMOD}/Connector_PinHeader_2.54mm.3dshapes/PinHeader_1x02_P2.54mm_Vertical.wrl
+      (at (xyz 0 0 0))
+      (scale (xyz 1 1 1))
+      (rotate (xyz 0 0 0))
+    )
+  )
   (module Package_DIP:DIP-24_W15.24mm (layer F.Cu)
     (at 194.8662 128.80746 180)
@@
       (net 1 "Net-(J1-Pad22)"))
     (model ${KISYS3DMOD}/Package_DIP.3dshapes/DIP-24_W15.24mm.wrl
-      (at (xyz 0 0 0))
-      (scale (xyz 1 1 1))
-      (rotate (xyz 0 0 0))
-    )
-  )
-  (module Connector_PinHeader_2.54mm:PinHeader_1x02_P2.54mm_Vertical (layer F.Cu)
-    (at 208.7262 132.76746)
-    (descr "Through hole straight pin header, 1x02, 2.54mm pitch, single row")
-    (tags "Through hole pin header THT 1x02 2.54mm single row")
-    (fp_text reference T1 (at 0 -2.33) (layer F.SilkS)
-      (effects (font (size 1 1) (thickness 0.15)))
-    )
-    (fp_text value Jumper (at 0 4.87) (layer F.Fab)
-      (effects (font (size 1 1) (thickness 0.15)))
-    )
-    (fp_line (start -0.635 -1.27) (end 1.27 -1.27) (layer F.Fab) (width 0.1))
-    (fp_line (start 1.27 -1.27) (end 1.27 3.81) (layer F.Fab) (width 0.1))
-    (fp_line (start 1.27 3.81) (end -1.27 3.81) (layer F.Fab) (width 0.1))
-    (fp_line (start -1.27 3.81) (end -1.27 -0.635) (layer F.Fab) (width 0.1))
-    (fp_line (start -1.27 -0.635) (end -0.635 -1.27) (layer F.Fab) (width 0.1))
-    (fp_line (start -1.33 3.87) (end 1.33 3.87) (layer F.SilkS) (width 0.12))
-    (fp_line (start -1.33 1.27) (end -1.33 3.87) (layer F.SilkS) (width 0.12))
-    (fp_line (start 1.33 1.27) (end 1.33 3.87) (layer F.SilkS) (width 0.12))
-    (fp_line (start -1.33 1.27) (end 1.33 1.27) (layer F.SilkS) (width 0.12))
-    (fp_line (start -1.33 0) (end -1.33 -1.33) (layer F.SilkS) (width 0.12))
-    (fp_line (start -1.33 -1.33) (end 0 -1.33) (layer F.SilkS) (width 0.12))
-    (fp_line (start -1.8 -1.8) (end -1.8 4.35) (layer F.CrtYd) (width 0.05))
-    (fp_line (start -1.8 4.35) (end 1.8 4.35) (layer F.CrtYd) (width 0.05))
-    (fp_line (start 1.8 4.35) (end 1.8 -1.8) (layer F.CrtYd) (width 0.05))
-    (fp_line (start 1.8 -1.8) (end -1.8 -1.8) (layer F.CrtYd) (width 0.05))
-    (fp_text user %R (at 0 1.27 90) (layer F.Fab)
-      (effects (font (size 1 1) (thickness 0.15)))
-    )
-    (pad 1 thru_hole rect (at 0 0) (size 1.7 1.7) (drill 1) (layers *.Cu *.Mask)
-      (net 46 "Net-(T1-Pad1)"))
-    (pad 2 thru_hole oval (at 0 2.54) (size 1.7 1.7) (drill 1) (layers *.Cu *.Mask)
-      (net 44 /T))
-    (model ${KISYS3DMOD}/Connector_PinHeader_2.54mm.3dshapes/PinHeader_1x02_P2.54mm_Vertical.wrl
       (at (xyz 0 0 0))
       (scale (xyz 1 1 1))
@@
       (net 42 "Net-(J1-PadZ)"))
   )
+  (gr_text "S Address\nto U1" (at 174.5262 135.85746) (layer F.SilkS)
+    (effects (font (size 1 1) (thickness 0.15)))
+  )
+  (gr_text "T Address\nto U2" (at 123.0262 136.35746) (layer F.SilkS)
+    (effects (font (size 1 1) (thickness 0.15)))
+  )
   (gr_text "2732 EPROM" (at 186.9462 99.10746) (layer F.SilkS)
     (effects (font (size 1 1) (thickness 0.15)))
@@
     (effects (font (size 1 1) (thickness 0.15)))
   )
-  (gr_text "Apple-1\nEPROM Card" (at 123.5862 132.76746) (layer F.SilkS)
+  (gr_text "Apple-1\nEPROM Card" (at 163.0262 103.85746) (layer F.SilkS)
     (effects (font (size 1.5 1.5) (thickness 0.3)))
   )
@@
   (segment (start 169.16 141.04) (end 169.16 135.34126) (width 0.25) (layer F.Cu) (net 43))
   (segment (start 208.76 135.34126) (end 208.7262 135.30746) (width 0.25) (layer F.Cu) (net 44))
-  (segment (start 208.76 141.04) (end 208.76 135.34126) (width 0.25) (layer F.Cu) (net 44))
+  (via (at 208.7762 117.60746) (size 0.8) (drill 0.4) (layers F.Cu B.Cu) (net 44))
+  (segment (start 208.76 117.62366) (end 208.7762 117.60746) (width 0.25) (layer F.Cu) (net 44))
+  (segment (start 208.76 141.04) (end 208.76 117.62366) (width 0.25) (layer F.Cu) (net 44))
+  (segment (start 116.351199 133.972459) (end 117.5262 135.14746) (width 0.25) (layer B.Cu) (net 44))
+  (segment (start 129.166199 98.182459) (end 116.351199 110.997459) (width 0.25) (layer B.Cu) (net 44))
+  (segment (start 205.498201 98.182459) (end 129.166199 98.182459) (width 0.25) (layer B.Cu) (net 44))
+  (segment (start 116.351199 110.997459) (end 116.351199 133.972459) (width 0.25) (layer B.Cu) (net 44))
+  (segment (start 208.7762 101.460458) (end 205.498201 98.182459) (width 0.25) (layer B.Cu) (net 44))
+  (segment (start 208.7762 117.60746) (end 208.7762 101.460458) (width 0.25) (layer B.Cu) (net 44))
   (segment (start 179.6262 118.64746) (end 177.0462 121.22746) (width 0.25) (layer B.Cu) (net 45))
   (via (at 177.0462 132.76746) (size 0.8) (drill 0.4) (layers F.Cu B.Cu) (net 45))
@@
   (segment (start 177.0462 121.22746) (end 177.0462 124.84746) (width 0.25) (layer B.Cu) (net 45))
   (segment (start 177.0462 132.76746) (end 169.1262 132.76746) (width 0.25) (layer F.Cu) (net 45))
-  (segment (start 208.7262 132.76746) (end 208.7262 99.10746) (width 0.25) (layer B.Cu) (net 46))
-  (segment (start 207.801199 98.182459) (end 126.491201 98.182459) (width 0.25) (layer B.Cu) (net 46))
-  (segment (start 208.7262 99.10746) (end 207.801199 98.182459) (width 0.25) (layer B.Cu) (net 46))
-  (segment (start 126.491201 98.182459) (end 117.6462 107.02746) (width 0.25) (layer B.Cu) (net 46))
-  (segment (start 117.6462 107.02746) (end 117.6462 114.94746) (width 0.25) (layer B.Cu) (net 46))
-  (via (at 123.5862 120.88746) (size 0.8) (drill 0.4) (layers F.Cu B.Cu) (net 46))
-  (segment (start 117.6462 114.94746) (end 123.5862 120.88746) (width 0.25) (layer B.Cu) (net 46))
-  (segment (start 125.8262 118.64746) (end 128.1462 118.64746) (width 0.25) (layer F.Cu) (net 46))
-  (segment (start 123.5862 120.88746) (end 125.8262 118.64746) (width 0.25) (layer F.Cu) (net 46))
+  (via (at 124.2762 118.60746) (size 0.8) (drill 0.4) (layers F.Cu B.Cu) (net 46))
+  (segment (start 117.5262 125.35746) (end 124.2762 118.60746) (width 0.25) (layer B.Cu) (net 46))
+  (segment (start 117.5262 132.60746) (end 117.5262 125.35746) (width 0.25) (layer B.Cu) (net 46))
+  (segment (start 128.1062 118.60746) (end 128.1462 118.64746) (width 0.25) (layer F.Cu) (net 46))
+  (segment (start 124.2762 118.60746) (end 128.1062 118.60746) (width 0.25) (layer F.Cu) (net 46))
 )
